File: Adapterboard.kicad_pcb (KiCad board)
At the start: 2 copper layers, 100 x 100 mm, 72 parts, among them J101 Conn_01x01_Pin, J102 Conn_01x01_Pin, J103 JTAG, J104 Conn_01x01_Pin, J105 TUNNEL_IN, J106 Power in +15V, J107 Power in -15V, J108 Power out Preamplifier, J109 Piezo, J110 TUNNEL_1, J111 USB_Connector, U101 ADS1115A, U102 DAC X, U103 ESP32-DEVKITC-32D, U104 DAC Y, U106 DAC Z, U107 ADC 8 Click, U108 mint, U109 UniRegensburg, U110 OTH, U201 TL072, U301 TL072

Commit message: pcb-supermarkt
Parts:
- D103: value LED_RED -> RED
- D104: value LED_YELLOW -> YELLOW
- D105: value LED_GREEN -> GREEN
- J101, J102, J104: value Conn_01x01_Pin -> 1xPin
- J103: value JTAG -> JTAG(optional)
- J110: value TUNNEL_1 -> 2xPin
- U101: value ADS1115A -> ADS1115A(optional)
Other:
- board text added: "ADS1115 ADC Modul(optional)"
- board text added: "TUNNEL amp VCC"
- board text removed: "2*Pin"
- board text removed: "Adafruit ADS1115 (optional)"
- board text removed: "TUNNEL VCC"
