File: Adapterboard.kicad_pcb (KiCad board)
At the start: 2 copper layers, 100 x 100 mm, 72 parts, among them J101 1xPin, J102 1xPin, J103 JTAG(optional), J104 1xPin, J105 TUNNEL_IN, J106 Power in +15V, J107 Power in -15V, J108 Power out Preamplifier, J109 Piezo, J110 2xPin, J111 USB_Connector, U101 ADS1115A(optional), U102 DAC X, U103 ESP32-DEVKITC-32D, U104 DAC Y, U106 DAC Z, U107 ADC 8 Click, U108 mint, U109 UniRegensburg, U110 OTH, U201 TL072, U301 TL072

Commit message: Added backup folder from 3.0. Added gerber files
Other:
- board text added: "500 € STM Ver 3.0.1 JAN 2026"
- board text removed: "500 € STM Ver 3.0 FEB 2025"
Changed lines of the file:
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@@
 	(title_block
 		(title "500 EUR STM Adapterboard")
-		(date "2025-02-18")
-		(rev "3.0")
+		(date "2026-01-19")
+		(rev "3.0.1")
 		(company "Univerität Regensburg")
 	)
@@
 		(tenting front back)
 		(pcbplotparams
-			(layerselection 0x00000000_00000000_55555555_5755f5ff)
-			(plot_on_all_layers_selection 0x00000000_00000000_00000000_00000000)
+			(layerselection 0x00000000_00000000_5555555f_ff5d557f)
+			(plot_on_all_layers_selection 0x00000000_00000000_0000000a_aa08002f)
 			(disableapertmacros no)
 			(usegerberextensions no)
@@
 			(outputformat 1)
 			(mirror no)
-			(drillshape 1)
+			(drillshape 0)
 			(scaleselection 1)
-			(outputdirectory "")
+			(outputdirectory "Production/")
 		)
 	)
@@
 		)
 	)
-	(gr_text "500 € STM\nVer 3.0 FEB 2025"
+	(gr_text "500 € STM\nVer 3.0.1 JAN 2026"
 		(at 58.42 147.955 0)
 		(layer "F.SilkS")
