File: Adapterboard.kicad_sch (KiCad schematic)
At the start: 72 parts, among them J101 Conn_01x01_Pin, J102 Conn_01x01_Pin, J103 JTAG, J104 Conn_01x01_Pin, J105 TUNNEL_IN, J106 Power in +15V, J107 Power in -15V, J108 Power out Preamplifier, J109 Piezo, J110 TUNNEL_1, J111 USB_Connector, U101 ADS1115A, U102 DAC X, U103 ESP32-DEVKITC-32D, U104 DAC Y, U106 DAC Z, U107 ADC 8 Click, U108 mint, U109 UniRegensburg, U110 OTH, U201 TL072, U301 TL072

Commit message: pcb-supermarkt
Parts:
- D103: value LED_RED -> RED
- D104: value LED_YELLOW -> YELLOW
- D105: value LED_GREEN -> GREEN
- J101, J102, J104: value Conn_01x01_Pin -> 1xPin
- J103: value JTAG -> JTAG(optional)
- J110: value TUNNEL_1 -> 2xPin
- U101: value ADS1115A -> ADS1115A(optional)
Other:
- note added: "Alternative TUNNEL ADC. Do not mount"
- note removed: "optional"
- moved on the sheet: U101
Changed lines of the file:
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@@
 	)
 	(no_connect
-		(at 350.52 179.07)
+		(at 373.38 184.15)
 	)
 	(no_connect
@@
 	)
 	(no_connect
-		(at 350.52 181.61)
+		(at 373.38 186.69)
 	)
 	(no_connect
@@
 	)
 	(no_connect
-		(at 372.11 170.18)
+		(at 394.97 175.26)
 	)
 	(no_connect
@@
 	)
 	(no_connect
-		(at 350.52 184.15)
+		(at 373.38 189.23)
 	)
 	(no_connect
@@
 	(wire
 		(pts
-			(xy 360.68 195.58) (xy 360.68 198.12)
+			(xy 383.54 200.66) (xy 383.54 203.2)
 		)
 		(stroke
@@
 	(wire
 		(pts
-			(xy 340.36 186.69) (xy 350.52 186.69)
+			(xy 363.22 191.77) (xy 373.38 191.77)
 		)
 		(stroke
@@
 	(wire
 		(pts
-			(xy 340.36 172.72) (xy 350.52 172.72)
+			(xy 363.22 177.8) (xy 373.38 177.8)
 		)
 		(stroke
@@
 	(wire
 		(pts
-			(xy 340.36 170.18) (xy 350.52 170.18)
+			(xy 363.22 175.26) (xy 373.38 175.26)
 		)
 		(stroke
@@
 	(wire
 		(pts
-			(xy 344.17 175.26) (xy 350.52 175.26)
+			(xy 367.03 180.34) (xy 373.38 180.34)
 		)
 		(stroke
@@
 	(wire
 		(pts
-			(xy 360.68 158.75) (xy 360.68 162.56)
+			(xy 383.54 163.83) (xy 383.54 167.64)
 		)
 		(stroke
@@
 		)
 	)
-	(text "optional"
-		(exclude_from_sim no)
-		(at 148.59 64.77 0)
-		(effects
-			(font
-				(size 1.27 1.27)
-			)
-			(justify left bottom)
-		)
-	)
 	(text "Powersupply +-15V in and \nPreamplifier out"
 		(exclude_from_sim no)
@@
 		)
 	)
+	(text "Alternative TUNNEL ADC. \nDo not mount"
+		(exclude_from_sim no)
+		(at 345.44 160.02 0)
+		(effects
+			(font
+				(size 2.54 2.54)
+				(thickness 0.508)
+				(bold yes)
+			)
+			(justify left bottom)
+		)
+	)
 	(text "Z-X"
 		(exclude_from_sim no)
@@
 	(global_label "ESP32_SCL"
 		(shape input)
-		(at 340.36 170.18 180)
+		(at 363.22 175.26 180)
 		(fields_autoplaced yes)
 		(effects
@@
 		)
 		(property "Intersheetrefs" "${INTERSHEET_REFS}"
-			(at 326.8521 170.18 0)
+			(at 349.7121 175.26 0)
 			(effects
 				(font
@@
 	(global_label "TUNNEL_TO_ADC_A3"
 		(shape input)
-		(at 340.36 186.69 180)
+		(at 363.22 191.77 180)
 		(fields_autoplaced yes)
 		(effects
@@
 		)
 		(property "Intersheetrefs" "${INTERSHEET_REFS}"
-			(at 319.111 186.69 0)
+			(at 341.971 191.77 0)
 			(effects
 				(font
@@
 	(global_label "ESP32_SDA"
 		(shape input)
-		(at 340.36 172.72 180)
+		(at 363.22 177.8 180)
 		(fields_autoplaced yes)
 		(effects
@@
 		)
 		(property "Intersheetrefs" "${INTERSHEET_REFS}"
-			(at 326.7916 172.72 0)
+			(at 349.6516 177.8 0)
 			(effects
 				(font
@@
 			)
 		)
-		(property "Description" ""
+		(property "Description" "MIKROE DAC 2 CLICK 16 bit DAC wirh LTC2601"
 			(at 53.34 118.11 0)
 			(effects
@@
 			)
 		)
-		(property "Description" ""
+		(property "Description" "MIKROE DAC 2 CLICK 16 bit DAC wirh LTC2601"
 			(at 176.53 118.11 0)
 			(effects
@@
 			)
 		)
-		(property "Description" ""
+		(property "Description" "MICROE ADC 8 CLICK 16 bit with ADS1115"
 			(at 300.99 116.84 0)
 			(effects
@@
 			)
 		)
-		(property "Datasheet" "~"
+		(property "Datasheet" "https://www.reichelt.de/de/de/shop/produkt/leiterplattenklemme_2_polig_rm_2_54_mm-276214?PROVID=2788&gad_source=1&gclid=Cj0KCQiAwtu9BhC8ARIsAI9JHal5xTnKnBgdLY6WmmCnl3_esX6RiSlgn1cEoWoG2r5Xr17Bj39ZyN8aAlpDEALw_wcB"
 			(at 241.3 43.18 0)
 			(effects
@@
 			)
 		)
-		(property "Description" "Generic screw terminal, single row, 01x02, script generated (kicad-library-utils/schlib/autogen/connector/)"
+		(property "Description" "PCB terminal block 2.54 mm"
 			(at 241.3 43.18 0)
 			(effects
@@
 			)
 		)
-		(property "Description" ""
+		(property "Description" "MIKROE DAC 2 CLICK 16 bit DAC wirh LTC2601"
 			(at 114.3 118.11 0)
 			(effects
@@
 			)
 		)
-		(property "Value" "TUNNEL_1"
+		(property "Value" "2xPin"
 			(at 294.005 95.25 0)
 			(effects
@@
 			)
 		)
-		(property "Datasheet" "~"
+		(property "Datasheet" "https://www.reichelt.de/de/de/shop/produkt/leiterplattenklemme_5_polig_rm_2_54_mm-276217"
 			(at 279.4 205.74 0)
 			(effects
@@
 			)
 		)
-		(property "Description" "Generic screw terminal, single row, 01x05, script generated (kicad-library-utils/schlib/autogen/connector/)"
+		(property "Description" "PCB terminal block 2.54 mm"
 			(at 279.4 205.74 0)
 			(effects
@@
 			)
 		)
-		(property "Value" "LED_GREEN"
+		(property "Value" "GREEN"
 			(at 149.352 49.276 0)
 			(effects
@@
 			)
 		)
-		(property "Value" "Conn_01x01_Pin"
+		(property "Value" "1xPin"
 			(at 109.855 102.87 0)
 			(effects
@@
 	(symbol
 		(lib_id "power:GND")
-		(at 360.68 198.12 0)
+		(at 383.54 203.2 0)
 		(unit 1)
 		(exclude_from_sim no)
@@
 		(dnp no)
 		(property "Reference" "#PWR0156"
-			(at 360.68 204.47 0)
+			(at 383.54 209.55 0)
 			(effects
 				(font
@@
 		)
 		(property "Value" "GND"
-			(at 360.807 202.5142 0)
+			(at 383.667 207.5942 0)
 			(effects
 				(font
@@
 		)
 		(property "Footprint" ""
-			(at 360.68 198.12 0)
+			(at 383.54 203.2 0)
 			(effects
 				(font
@@
 		)
 		(property "Datasheet" ""
-			(at 360.68 198.12 0)
+			(at 383.54 203.2 0)
 			(effects
 				(font
@@
 		)
 		(property "Description" ""
-			(at 360.68 198.12 0)
+			(at 383.54 203.2 0)
 			(effects
 				(font
@@
 	(symbol
 		(lib_id "power:+5V")
-		(at 360.68 158.75 0)
+		(at 383.54 163.83 0)
 		(unit 1)
 		(exclude_from_sim no)
@@
 		(dnp no)
 		(property "Reference" "#PWR0155"
-			(at 360.68 162.56 0)
+			(at 383.54 167.64 0)
 			(effects
 				(font
@@
 		)
 		(property "Value" "+5V"
-			(at 361.061 155.4988 90)
+			(at 383.921 160.5788 90)
 			(effects
 				(font
@@
 		)
 		(property "Footprint" ""
-			(at 360.68 158.75 0)
+			(at 383.54 163.83 0)
 			(effects
 				(font
@@
 		)
 		(property "Datasheet" ""
-			(at 360.68 158.75 0)
+			(at 383.54 163.83 0)
 			(effects
 				(font
@@
 		)
 		(property "Description" ""
-			(at 360.68 158.75 0)
+			(at 383.54 163.83 0)
 			(effects
 				(font
@@
 			)
 		)
-		(property "Value" "Conn_01x01_Pin"
+		(property "Value" "1xPin"
 			(at 170.18 104.14 0)
 			(effects
@@
 			)
 		)
-		(property "Datasheet" "~"
+		(property "Datasheet" "https://www.reichelt.de/de/de/shop/produkt/leiterplattenklemme_2_polig_rm_2_54_mm-276214?PROVID=2788&gad_source=1&gclid=Cj0KCQiAwtu9BhC8ARIsAI9JHal5xTnKnBgdLY6WmmCnl3_esX6RiSlgn1cEoWoG2r5Xr17Bj39ZyN8aAlpDEALw_wcB"
 			(at 241.3 35.56 0)
 			(effects
@@
 			)
 		)
-		(property "Description" "Generic screw terminal, single row, 01x02, script generated (kicad-library-utils/schlib/autogen/connector/)"
+		(property "Description" "PCB terminal block 2.54 mm"
 			(at 241.3 35.56 0)
 			(effects
@@
 			)
 		)
-		(property "Datasheet" "~"
+		(property "Datasheet" "https://www.reichelt.de/de/de/shop/produkt/leiterplattenklemme_2_polig_rm_2_54_mm-276214?PROVID=2788&gad_source=1&gclid=Cj0KCQiAwtu9BhC8ARIsAI9JHal5xTnKnBgdLY6WmmCnl3_esX6RiSlgn1cEoWoG2r5Xr17Bj39ZyN8aAlpDEALw_wcB"
 			(at 222.25 101.6 0)
 			(effects
@@
 			)
 		)
-		(property "Description" ""
+		(property "Description" "PCB terminal block 2.54 mm"
 			(at 222.25 101.6 0)
 			(effects
@@
 	(symbol
 		(lib_id "My_Library:ADS1115_ADC_module")
-		(at 360.68 179.07 0)
+		(at 383.54 184.15 0)
 		(unit 1)
 		(exclude_from_sim no)
@@
 		(fields_autoplaced yes)
 		(property "Reference" "U101"
-			(at 373.38 165.1314 0)
+			(at 396.24 170.2114 0)
 			(effects
 				(font
@@
 			)
 		)
-		(property "Value" "ADS1115A"
-			(at 361.95 183.134 0)
+		(property "Value" "ADS1115A(optional)"
+			(at 384.81 188.214 0)
 			(effects
 				(font
@@
 		)
 		(property "Footprint" "Connector_PinHeader_2.54mm:PinHeader_1x10_P2.54mm_Vertical"
-			(at 360.68 179.07 0)
+			(at 383.54 184.15 0)
 			(show_name yes)
 			(effects
@@
 			)
 		)
-		(property "Datasheet" ""
-			(at 360.68 179.07 0)
+		(property "Datasheet" "https://www.az-delivery.de/products/analog-digitalwandler-ads1115-mit-i2c-interface"
+			(at 383.54 184.15 0)
 			(effects
 				(font
@@
 			)
 		)
-		(property "Description" ""
-			(at 360.68 179.07 0)
+		(property "Description" "ADS1115 ADC Modul"
+			(at 383.54 184.15 0)
 			(effects
 				(font
@@
 			)
 		)
-		(property "Datasheet" "~"
+		(property "Datasheet" "https://www.reichelt.de/de/de/shop/produkt/leiterplattenklemme_3_polig_rm_2_54_mm-276215"
 			(at 241.3 73.66 0)
 			(effects
@@
 			)
 		)
-		(property "Description" "Generic screw terminal, single row, 01x03, script generated (kicad-library-utils/schlib/autogen/connector/)"
+		(property "Description" "PCB terminal block 2.54 mm"
 			(at 241.3 73.66 0)
 			(effects
@@
 			)
 		)
-		(property "Value" "JTAG"
+		(property "Value" "JTAG(optional)"
 			(at 142.875 66.04 0)
 			(effects
@@
 			)
 		)
-		(property "Description" ""
+		(property "Description" "JTAG Connector for Debbugging ESP"
 			(at 142.24 73.66 0)
 			(effects
@@
 	(symbol
 		(lib_id "power:GND")
-		(at 344.17 175.26 0)
+		(at 367.03 180.34 0)
 		(unit 1)
 		(exclude_from_sim no)
@@
 		(dnp no)
 		(property "Reference" "#PWR0157"
-			(at 344.17 181.61 0)
+			(at 367.03 186.69 0)
 			(effects
 				(font
@@
 		)
 		(property "Value" "GND"
-			(at 344.297 179.6542 0)
+			(at 367.157 184.7342 0)
 			(effects
 				(font
@@
 		)
 		(property "Footprint" ""
-			(at 344.17 175.26 0)
+			(at 367.03 180.34 0)
 			(effects
 				(font
@@
 		)
 		(property "Datasheet" ""
-			(at 344.17 175.26 0)
+			(at 367.03 180.34 0)
 			(effects
 				(font
@@
 		)
 		(property "Description" ""
-			(at 344.17 175.26 0)
+			(at 367.03 180.34 0)
 			(effects
 				(font
@@
 			)
 		)
-		(property "Value" "LED_RED"
+		(property "Value" "RED"
 			(at 148.336 38.862 0)
 			(effects
@@
 			)
 		)
-		(property "Value" "Conn_01x01_Pin"
+		(property "Value" "1xPin"
 			(at 46.355 102.87 0)
 			(effects
@@
 			)
 		)
-		(property "Value" "LED_YELLOW"
+		(property "Value" "YELLOW"
 			(at 150.114 43.942 0)
 			(effects
